Commit message: ur5.xacro chage
added world link to get correct orentation of robot stand

File: catkin_ws/src/fmauch_universal_robot/ur_description/urdf/ur5.xacro (robot description, xacro)
@@ -14,4 +14,8 @@
     Refer to 'inc/ur_macro.xacro' for more information.
  #   -->
+ <!--world link is added -->
+<link name="world">
+</link>
+<!--Tool link is added -->
 <link name="tool">
   <visual>
@@ -27,4 +31,5 @@
    <origin rpy="0 0 0" xyz="0 0 0"/>
 </link>
+<!--Table link is added -->
 <link name="table">
   <origin rpy="-1.5708 0 0" xyz="0 0 0"/>
@@ -40,5 +45,9 @@
   </collision>
 </link>
-0
+<joint name="world_to_table" type="fixed">
+  <parent link="world"/>
+  <child link="table"/>
+  <origin xyz="0 0 0" rpy="1.5708 0 0"/>
+</joint>
 <joint name="table_to_robot" type="fixed">
   <parent link="table"/>

Commit message: catkin_chages

File: catkin_ws/src/fmauch_universal_robot/ur_description/urdf/ur5.xacro (robot description, xacro)
@@ -21,10 +21,10 @@
   <visual>
     <geometry>
-       <mesh filename="package://ur5uia/meshes/finaltool.STL" scale="0.001 0.001 0.001"/>
+       <mesh filename="package://ur_description/meshes/ur5/collision/finaltool.STL" scale="0.001 0.001 0.001"/>
     </geometry>
   </visual>
   <collision>
     <geometry>
-      <mesh filename="package://ur5uia/meshes/finaltool.dae" scale="0.001 0.001 0.001"/>
+      <mesh filename="package://ur_description/meshes/ur5/visual/finaltool.dae" scale="0.001 0.001 0.001"/>
     </geometry>
   </collision>
@@ -36,10 +36,10 @@
   <visual>
     <geometry>
-       <mesh filename="package://ur5uia/meshes/table.STL" scale="0.001 0.001 0.001" rpy= "-1.5708 0 0"/>
+       <mesh filename="package://ur_description/meshes/ur5/collision/table.STL" scale="0.001 0.001 0.001" rpy= "-1.5708 0 0"/>
     </geometry>
   </visual>
   <collision>
     <geometry>
-      <mesh filename="package://ur5uia/meshes/table.dae" scale="0.001 0.001 0.001" origin= "-1.5708 0 0"/>
+      <mesh filename="package://ur_description/meshes/ur5/visual/table.dae" scale="0.001 0.001 0.001" origin= "-1.5708 0 0"/>
     </geometry>
   </collision>
